File: CBMINI.sch (EAGLE design)
At the start: 59 parts, among them IC1 ATMEGA32U4NT-TQFP, IC2 MCP2515, IC3 MCP2551, J1 USB-B-PTH, X1 INPUT, X2 OUTPUT

Commit message: Isolation diodes between CAN and chair power, and switched parts to SuperHouse libraries for v2.3 release
Parts:
- removed JP2: PWR, SuperHouse-Connectors:M02-PIN
- added D2, D3: SS56, SuperHouse-DiscreteSemi:DIODESMA
- D1: value 1N4004 -> SS56
- S2: device freetronics-jon:SWITCH-DPDT3 -> SuperHouse-Switches:SWITCH-DPDT3
- X1: device SparkFun-Connectors:DB9MALE -> SuperHouse-Connectors:DB9-PCB-PLUG
- X2: device SparkFun-Connectors:DB9FEMALE -> SuperHouse-Connectors:DB9-PCB-SOCKET
Connections:
- net 12V: now also D2.A; no longer JP2.2
- net 24V: now also D3.C
- net VREF: now also D2.C, D3.A; no longer JP2.1
Other:
- note added: "(C)2018-2020 SuperHouse Automation: www.superhouse.tv"
- note added: "V2.3 (2020-02-18)"
- note removed: "(C)2018-2019 SuperHouse Automation: www.superhouse.tv"
- note removed: "Power strategy: 1. Connected to Permobil. Accept reference voltage, pass it through. Jumper off. 2. Connected to WMC. Take 24V on CAN, generate reference voltage. Jumper on."
- note removed: "V2.2 (2019-11-13)"
- moved on the sheet: C10, C11, REG2
